Commit message: Add measured frame and utility functions

File: models/object_3d/se3_object.urdf (robot description, URDF)
Before this commit: robot obj_se3, 5 links, 4 joints
Joints:
- removed joint measured_com_joint
- added joint com_measured_joint: type fixed, parent obj_com, child obj_measured, origin xyz=0 0 0 rpy=0 0 0
